Commit message: 更新urdf文件

File: genimind_description/urdf/genimind_description.urdf (robot description, URDF)
Before this commit: robot genimind_description, 9 links, 8 joints
Joints:
- joint base_joint: origin xyz=-0.000168546343865929 0.000259630628177465 0.057 rpy=0 0 0 -> xyz=0.0 0.0 0.057 rpy=0 0 0
